File: klepcbgen/left-conn.kicad_sch (KiCad schematic)
At the start: 19 parts, among them J3 USB_C_Plug, J4 USB_C_Receptacle

Commit message: Continuing.
Connections:
- net COMMON_COLUMN is gone; now on net COL6: JP6.2 (C)
- net COL10: now also JP10.2 (C); no longer JP11.2 (C)
- net COL11: now also JP11.2 (C); no longer JP12.2 (C)
- net COL12: now also JP12.2 (C); no longer JP13.2 (C)
- net COL13: now also JP13.2 (C); no longer JP14.2 (C)
- net COL14: now also JP14.2 (C); no longer JP15.2 (C)
- net COL6: no longer JP7.2 (C)
- net COL7: now also JP7.2 (C); no longer JP8.2 (C)
- net COL8: now also JP8.2 (C); no longer JP9.2 (C)
- net COL9: now also JP9.2 (C); no longer JP10.2 (C)
