File: pcb/69split.kicad_sch (KiCad schematic)
At the start: 0 parts

Commit message: Figured out what GPIOs to use.
Other:
- note added: "69SPLIT KEYBOARD"
- note removed: "69SPLIT SWEYBOARD"
Changed lines of the file:
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@@
 		)
 	)
-	(text "69SPLIT SWEYBOARD"
+	(text "69SPLIT KEYBOARD"
 		(exclude_from_sim no)
 		(at 142.24 38.1 0)

Commit message: I think schematic is done?
Other:
- title: Split Normal 69 -> 69SPLIT KEYBOARD
Changed lines of the file:
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@@
 	(paper "A4")
 	(title_block
-		(title "Split Normal 69")
+		(title "69SPLIT KEYBOARD")
 		(date "2025-06-11")
 	)
