File: pcb/atmega32u4.kicad_sch (KiCad schematic)
At the start: 13 parts, among them J2 Conn_02x03_Odd_Even, SW1 RESET_SW, U1 ATmega32U4-AU, Y1 Crystal

Commit message: Added MPNs and footprints for I think everything.
Parts:
- C1, C3, C4, C8, C9: footprint Capacitor_SMD:C_0805_2012Metric_Pad1.15x1.40mm_HandSolder -> Capacitor_SMD:C_0603_1608Metric_Pad1.08x0.95mm_HandSolder; MPN (none) -> Generic; Rating (none) -> 10V
- C6, C7: value 22p -> 30p; footprint Capacitor_SMD:C_0805_2012Metric_Pad1.15x1.40mm_HandSolder -> Capacitor_SMD:C_0603_1608Metric_Pad1.08x0.95mm_HandSolder; MPN (none) -> CC0603JRNPO0BN300; Rating (none) -> 10V
- J2: MPN (none) -> Generic
- R1, R4: footprint Resistor_SMD:R_0805_2012Metric_Pad1.15x1.40mm_HandSolder -> Resistor_SMD:R_0603_1608Metric_Pad0.98x0.95mm_HandSolder; MPN (none) -> Generic
- SW1: footprint Button_Switch_SMD:SW_Push_1P1T_NO_6x6mm_H9.5mm -> Button_Switch_THT:SW_PUSH-12mm_Wuerth-430476085716; MPN (none) -> 430476085716
- U1: MPN (none) -> ATMEGA32U4-AUR
- Y1: footprint Crystal:Crystal_SMD_5032-2Pin_5.0x3.2mm_HandSoldering -> Crystal:Crystal_HC49-4H_Vertical; MPN (none) -> ABL-16.000MHz-B4Y; Rating (none) -> 16 MHz
Other:
- note added: "COL1 - SCK COL2 - MOSI COL3 - MISO"

Commit message: Continuing...no one will read this but me.
Parts:
- SW1: value RESET_SW -> SW_Push
- renumbered C3 to C2, C4 to C3, C1 to C4, C9 to C5, R1 to R5, R4 to R6
Other:
- note added: "ATMEGA32U4"
- note added: "COL1 - SCSW COL2 - MOSI COL3 - MISO"
- note removed: "COL1 - SCK COL2 - MOSI COL3 - MISO"
- moved on the sheet: C2, C3, C4, C5, C6, C7, C8, J2, R5, R6, SW1, U1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

Commit message: Figured out what GPIOs to use.
Connections:
- net COL0: now also U1.20 (PD2); no longer U1.8 (PB0)
- net COL1: now also U1.21 (PD3); no longer U1.9 (PB1)
- net COL10: now also U1.37 (PF6); no longer U1.25 (PD4)
- net COL11: now also U1.38 (PF5); no longer U1.36 (PF7)
- net COL12: now also U1.39 (PF4); no longer U1.37 (PF6)
- net COL13: now also U1.40 (PF1); no longer U1.38 (PF5)
- net COL14: now also U1.41 (PF0); no longer U1.39 (PF4)
- net COL2: now also U1.25 (PD4); no longer U1.10 (PB2)
- net COL3: now also U1.22 (PD5); no longer U1.11 (PB3)
- net COL4: now also U1.26 (PD6); no longer U1.12 (PB7)
- net COL5: now also U1.27 (PD7); no longer U1.18 (PD0)
- net COL6: now also U1.28 (PB4); no longer U1.19 (PD1)
- net COL7: now also U1.31 (PC6); no longer U1.20 (PD2)
- net COL8: now also U1.32 (PC7); no longer U1.21 (PD3)
- net COL9: now also U1.36 (PF7); no longer U1.22 (PD5)
- net ROW0: now also U1.9 (PB1); no longer U1.32 (PC7)
- net ROW1: now also U1.10 (PB2); no longer U1.31 (PC6)
- net ROW2: now also U1.11 (PB3); no longer U1.30 (PB6)
- net ROW3: now also U1.18 (PD0); no longer U1.29 (PB5)
- net ROW4: now also U1.19 (PD1); no longer U1.28 (PB4)
- net INDICATOR_GPIO: now reaches U1.1 (PE6)
- new net GPIO_OUT_PB5: U1.29 (PB5)
- new net GPIO_OUT_PB6: U1.30 (PB6)
- new net GPIO_OUT_PB7: U1.12 (PB7)
- new net INDICATOR_CAPS_LOCK: U1.8 (PB0)
- no-connect marks 6 -> 1
Other:
- moved on the sheet: R6

Commit message: I think schematic is done?
Parts:
- added R7, R8, R9: 330R, Resistor_SMD:R_0603_1608Metric_Pad0.98x0.95mm_HandSolder, symbol Device:R
Connections:
- net GPIO_OUT_PB5: now also R7.1; no longer U1.29 (PB5)
- net GPIO_OUT_PB6: now also R8.1; no longer U1.30 (PB6)
- net GPIO_OUT_PB7: now also R9.1; no longer U1.12 (PB7)
- new net: R9.2, U1.12 (PB7)
- new net: R7.2, U1.29 (PB5)
- new net: R8.2, U1.30 (PB6)
Other:
- note added: "330R for 10mA limit"
- title: Split Normal 69 -> 69SPLIT KEYBOARD
