File: pcb/gpio.kicad_sch (KiCad schematic)
At the start: 1 part, among them J4 Conn_01x03_Socket

Commit message: I think schematic is done?
Connections:
- net GPIO_OUT_PB5: now reaches J4.1 (Pin_1)
- net GPIO_OUT_PB6: now reaches J4.2 (Pin_2)
- net GPIO_OUT_PB7: now reaches J4.3 (Pin_3)
Other:
- note added: "GPIO OUTPUTS"
- title: Split Normal 69 -> 69SPLIT KEYBOARD
- moved on the sheet: J4
Changed lines of the file:
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@@
 	(paper "A4")
 	(title_block
-		(title "Split Normal 69")
+		(title "69SPLIT KEYBOARD")
 		(date "2025-06-11")
+	)
+	(text "GPIO OUTPUTS"
+		(exclude_from_sim no)
+		(at 142.494 35.052 0)
+		(effects
+			(font
+				(face "Book Antiqua")
+				(size 7.62 7.62)
+				(color 0 0 0 1)
+			)
+		)
+	)
+	(bus_entry
+		(at 115.57 93.98)
+		(size -2.54 2.54)
+		(stroke
+			(width 0)
+			(type default)
+		)
+	)
+	(bus_entry
+		(at 115.57 99.06)
+		(size -2.54 2.54)
+		(stroke
+			(width 0)
+			(type default)
+		)
+	)
+	(bus_entry
+		(at 115.57 96.52)
+		(size -2.54 2.54)
+		(stroke
+			(width 0)
+			(type default)
+		)
+	)
+	(bus
+		(pts
+			(xy 113.03 101.6) (xy 113.03 99.06)
+		)
+		(stroke
+			(width 0)
+			(type default)
+		)
+	)
+	(wire
+		(pts
+			(xy 115.57 93.98) (xy 171.45 93.98)
+		)
+		(stroke
+			(width 0)
+			(type default)
+		)
+	)
+	(wire
+		(pts
+			(xy 115.57 99.06) (xy 171.45 99.06)
+		)
+		(stroke
+			(width 0)
+			(type default)
+		)
+	)
+	(bus
+		(pts
+			(xy 113.03 99.06) (xy 113.03 96.52)
+		)
+		(stroke
+			(width 0)
+			(type default)
+		)
+	)
+	(bus
+		(pts
+			(xy 113.03 96.52) (xy 99.06 96.52)
+		)
+		(stroke
+			(width 0)
+			(type default)
+		)
+	)
+	(wire
+		(pts
+			(xy 115.57 96.52) (xy 171.45 96.52)
+		)
+		(stroke
+			(width 0)
+			(type default)
+		)
+	)
+	(label "GPIO_OUT_PB6"
+		(at 130.81 96.52 180)
+		(effects
+			(font
+				(size 1.27 1.27)
+			)
+			(justify right bottom)
+		)
+	)
+	(label "GPIO_OUT_PB7"
+		(at 130.81 99.06 180)
+		(effects
+			(font
+				(size 1.27 1.27)
+			)
+			(justify right bottom)
+		)
+	)
+	(label "GPIO_OUT_PB5"
+		(at 130.81 93.98 180)
+		(effects
+			(font
+				(size 1.27 1.27)
+			)
+			(justify right bottom)
+		)
+	)
+	(hierarchical_label "{GPIO_OUT}"
+		(shape input)
+		(at 99.06 96.52 180)
+		(effects
+			(font
+				(size 1.27 1.27)
+			)
+			(justify right)
+		)
 	)
 	(symbol
 		(lib_id "Connector:Conn_01x03_Socket")
-		(at 140.97 96.52 0)
+		(at 176.53 96.52 0)
 		(unit 1)
 		(exclude_from_sim no)
@@
 		(dnp no)
 		(fields_autoplaced yes)
-		(property "Reference" "J?"
-			(at 142.24 95.2499 0)
+		(property "Reference" "J4"
+			(at 177.8 95.2499 0)
 			(effects
 				(font
@@
 		)
 		(property "Value" "Conn_01x03_Socket"
-			(at 142.24 97.7899 0)
+			(at 177.8 97.7899 0)
 			(effects
 				(font
@@
 		)
 		(property "Footprint" "Connector_PinSocket_2.54mm:PinSocket_1x03_P2.54mm_Horizontal"
-			(at 140.97 96.52 0)
+			(at 176.53 96.52 0)
 			(effects
 				(font
@@
 		)
 		(property "Datasheet" "~"
-			(at 140.97 96.52 0)
+			(at 176.53 96.52 0)
 			(effects
 				(font
@@
 		)
 		(property "Description" "Generic connector, single row, 01x03, script generated"
-			(at 140.97 96.52 0)
+			(at 176.53 96.52 0)
 			(effects
 				(font
@@
 		)
 		(property "MPN" "Generic"
-			(at 140.97 96.52 0)
+			(at 176.53 96.52 0)
 			(effects
 				(font
