File: pcb/left-matrix.kicad_sch (KiCad schematic)
At the start: 58 parts, among them K69 Esc, K70 Tab, K71 Caps Lock, K72 Shift, K73 Ctrl, K74 !,1,,F1, K75 Q, K76 A, K77 Z, K78 Win, K79 @,2,,F2, K80 W, K81 S, K82 X, K83 Alt, K84 #,3,,F3, K85 E, K86 D, K87 C, K88 Space, K89 $,4,,F4, K90 R, K91 F, K92 V, K93 %,5,,F5, K94 T, K95 G, K96 B, K97 ^,6,,F6

Commit message: Added MPNs and footprints for I think everything.
Parts:
- K69, K70, K71, K72, K73, K74, K75, K76, K77, K78, K79, K80, K81, K82, K83, K84, K85, K86, K87, K88, K89, K90, K91, K92, K93, K94, K95, K96, K97: MPN (none) -> Generic

Commit message: Continuing...no one will read this but me.
Parts:
- renumbered D69 to D1, D80 to D10, D85 to D11, D90 to D12, D94 to D13, D71 to D14, D76 to D15, D81 to D16, D86 to D17, D91 to D18, D95 to D19, D74 to D2, D72 to D20, D77 to D21, D82 to D22, D87 to D23, D92 to D24, D96 to D25, D73 to D26, D78 to D27, D83 to D28, D88 to D29, D79 to D3, D84 to D4, D89 to D5, D93 to D6, D97 to D7, D70 to D8, D75 to D9, K75 to SW10, K80 to SW11, K85 to SW12, K90 to SW13, K94 to SW14, K71 to SW15, K76 to SW16, K81 to SW17, K86 to SW18, K91 to SW19, K69 to SW2, K95 to SW20, K72 to SW21, K77 to SW22, K82 to SW23, K87 to SW24, K92 to SW25, K96 to SW26, K73 to SW27, K78 to SW28, K83 to SW29, K74 to SW3, K88 to SW30, K79 to SW4, K84 to SW5, K89 to SW6, K93 to SW7, K97 to SW8, K70 to SW9
Other:
- note added: "LEFT MATRIX"

Commit message: I think schematic is done?
Other:
- title: Split Normal 69 -> 69SPLIT KEYBOARD
Changed lines of the file:
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@@
 	(paper "A4")
 	(title_block
-		(title "Split Normal 69")
+		(title "69SPLIT KEYBOARD")
 		(date "2025-06-11")
 	)
