File: pcb/right-matrix.kicad_sch (KiCad schematic)
At the start: 80 parts, among them SW31 &,7,,F7, SW32 *,8,,F8, SW33 (,9,,F9, SW34 ),0,,F10, SW35 _,-,,F11, SW36 +,=,,F12, SW37 Backspace, SW38 Delete,Insert, SW39 Y, SW40 U, SW41 I, SW42 O, SW43 P, SW44 {,[, SW45 },], SW46 |,\, SW47 ~~,`, SW48 H, SW49 J, SW50 K, SW51 L, SW52 :,;, SW53 ",', SW54 Enter, SW55 Home,PgUp, SW56 N, SW57 M, SW58 <,,, SW59 >,., SW60 ?,/, SW61 Shift, SW62 ↑, SW63 End,PgDn, SW64 Space, SW65 Alt, SW66 Fn, SW67 Ctrl, SW68 ←, SW69 ↓, SW70 →

Commit message: I think schematic is done?
Other:
- title: (none) -> 69SPLIT KEYBOARD
Changed lines of the file:
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@@
 	(generator_version "9.0")
 	(paper "A4")
+	(title_block
+		(title "69SPLIT KEYBOARD")
+		(date "2025-06-11")
+	)
 	(text "RIGHT MATRIX"
 		(exclude_from_sim no)
