File: pcb/right.kicad_sch (KiCad schematic)
At the start: 80 parts, among them K10 ),0,,F10, K11 _,-,,F11, K12 +,=,,F12, K13 Backspace, K14 Delete,Insert, K21 Y, K22 U, K23 I, K24 O, K25 P, K26 {,[, K27 },], K28 |,\, K29 ~~,`, K36 H, K37 J, K38 K, K39 L, K40 :,;, K41 ",', K42 Enter, K43 Home,PgUp, K50 N, K51 M, K52 <,,, K53 >,., K54 ?,/, K55 Shift, K56 ↑, K57 End,PgDn, K62 Space, K63 Alt, K64 Fn, K65 Ctrl, K66 ←, K67 ↓, K68 →, K7 &,7,,F7, K8 *,8,,F8, K9 (,9,,F9

Commit message: Added MPNs and footprints for I think everything.
Parts:
- K10, K11, K12, K13, K14, K21, K22, K23, K24, K25, K26, K27, K28, K29, K36, K37, K38, K39, K40, K41, K42, K43, K50, K51, K52, K53, K54, K55, K56, K57, K62, K63, K64, K65, K66, K67, K68, K7, K8, K9: MPN (none) -> Generic

Commit message: Continuing...no one will read this but me.
Parts:
- removed D10, D11, D12, D13, D14, D21, D22, D23, D24, D25, D26, D27, D28, D29, D36, D37, D38, D39, D40, D41, D42, D43, D50, D51, D52, D53, D54, D55, D56, D57, D62, D63, D64, D65, D66, D67, D68, D7, D8, D9: D, Diode_SMD:D_0805_2012Metric_Pad1.15x1.40mm_HandSolder, symbol Device:D
- removed K10: ),0,,F10, Button_Switch_Keyboard:SW_Cherry_MX_1.00u_PCB, symbol Switch:SW_Push
- removed K11: _,-,,F11, Button_Switch_Keyboard:SW_Cherry_MX_1.00u_PCB, symbol Switch:SW_Push
- removed K12: +,=,,F12, Button_Switch_Keyboard:SW_Cherry_MX_1.00u_PCB, symbol Switch:SW_Push
- removed K13: Backspace, Button_Switch_Keyboard:SW_Cherry_MX_2.00u_PCB, symbol Switch:SW_Push
- removed K14: Delete,Insert, Button_Switch_Keyboard:SW_Cherry_MX_1.00u_PCB, symbol Switch:SW_Push
- removed K21: Y, Button_Switch_Keyboard:SW_Cherry_MX_1.00u_PCB, symbol Switch:SW_Push
- removed K22: U, Button_Switch_Keyboard:SW_Cherry_MX_1.00u_PCB, symbol Switch:SW_Push
- removed K23: I, Button_Switch_Keyboard:SW_Cherry_MX_1.00u_PCB, symbol Switch:SW_Push
- removed K24: O, Button_Switch_Keyboard:SW_Cherry_MX_1.00u_PCB, symbol Switch:SW_Push
- removed K25: P, Button_Switch_Keyboard:SW_Cherry_MX_1.00u_PCB, symbol Switch:SW_Push
- removed K26: {,[, Button_Switch_Keyboard:SW_Cherry_MX_1.00u_PCB, symbol Switch:SW_Push
- removed K27: },], Button_Switch_Keyboard:SW_Cherry_MX_1.00u_PCB, symbol Switch:SW_Push
- removed K28: |,\, Button_Switch_Keyboard:SW_Cherry_MX_1.50u_PCB, symbol Switch:SW_Push
- removed K29: ~~,`, Button_Switch_Keyboard:SW_Cherry_MX_1.00u_PCB, symbol Switch:SW_Push
- removed K36: H, Button_Switch_Keyboard:SW_Cherry_MX_1.00u_PCB, symbol Switch:SW_Push
- removed K37: J, Button_Switch_Keyboard:SW_Cherry_MX_1.00u_PCB, symbol Switch:SW_Push
- removed K38: K, Button_Switch_Keyboard:SW_Cherry_MX_1.00u_PCB, symbol Switch:SW_Push
- removed K39: L, Button_Switch_Keyboard:SW_Cherry_MX_1.00u_PCB, symbol Switch:SW_Push
- removed K40: :,;, Button_Switch_Keyboard:SW_Cherry_MX_1.00u_PCB, symbol Switch:SW_Push
- removed K41: ",', Button_Switch_Keyboard:SW_Cherry_MX_1.00u_PCB, symbol Switch:SW_Push
- removed K42: Enter, Button_Switch_Keyboard:SW_Cherry_MX_2.25u_PCB, symbol Switch:SW_Push
- removed K43: Home,PgUp, Button_Switch_Keyboard:SW_Cherry_MX_1.00u_PCB, symbol Switch:SW_Push
- removed K50: N, Button_Switch_Keyboard:SW_Cherry_MX_1.00u_PCB, symbol Switch:SW_Push
- removed K51: M, Button_Switch_Keyboard:SW_Cherry_MX_1.00u_PCB, symbol Switch:SW_Push
- removed K52: <,,, Button_Switch_Keyboard:SW_Cherry_MX_1.00u_PCB, symbol Switch:SW_Push
- removed K53: >,., Button_Switch_Keyboard:SW_Cherry_MX_1.00u_PCB, symbol Switch:SW_Push
- removed K54: ?,/, Button_Switch_Keyboard:SW_Cherry_MX_1.00u_PCB, symbol Switch:SW_Push
- removed K55: Shift, Button_Switch_Keyboard:SW_Cherry_MX_1.75u_PCB, symbol Switch:SW_Push
- removed K56: ↑, Button_Switch_Keyboard:SW_Cherry_MX_1.00u_PCB, symbol Switch:SW_Push
- removed K57: End,PgDn, Button_Switch_Keyboard:SW_Cherry_MX_1.00u_PCB, symbol Switch:SW_Push
- removed K62: Space, Button_Switch_Keyboard:SW_Cherry_MX_2.75u_PCB, symbol Switch:SW_Push
- removed K63: Alt, Button_Switch_Keyboard:SW_Cherry_MX_1.00u_PCB, symbol Switch:SW_Push
- removed K64: Fn, Button_Switch_Keyboard:SW_Cherry_MX_1.00u_PCB, symbol Switch:SW_Push
- removed K65: Ctrl, Button_Switch_Keyboard:SW_Cherry_MX_1.00u_PCB, symbol Switch:SW_Push
- removed K66: ←, Button_Switch_Keyboard:SW_Cherry_MX_1.00u_PCB, symbol Switch:SW_Push
- removed K67: ↓, Button_Switch_Keyboard:SW_Cherry_MX_1.00u_PCB, symbol Switch:SW_Push
- removed K68: →, Button_Switch_Keyboard:SW_Cherry_MX_1.00u_PCB, symbol Switch:SW_Push
- removed K7: &,7,,F7, Button_Switch_Keyboard:SW_Cherry_MX_1.00u_PCB, symbol Switch:SW_Push
- removed K8: *,8,,F8, Button_Switch_Keyboard:SW_Cherry_MX_1.00u_PCB, symbol Switch:SW_Push
- removed K9: (,9,,F9, Button_Switch_Keyboard:SW_Cherry_MX_1.00u_PCB, symbol Switch:SW_Push
Other:
- added sheet Right Matrix (right-matrix.kicad_sch)
- sheet Right Keyboard Connector ports: added none; removed COMMON_COLUMN

Commit message: Figured out what GPIOs to use.
Other:
- added sheet GPIO Outputs (gpio.kicad_sch)
Changed lines of the file:
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@@
 		(date "2025-06-11")
 	)
+	(rectangle
+		(start 73.66 62.865)
+		(end 228.6 149.225)
+		(stroke
+			(width 0)
+			(type solid)
+			(color 255 43 5 1)
+		)
+		(fill
+			(type none)
+		)
+	)
 	(text "RIGHT KEYBOARD"
 		(exclude_from_sim no)
-		(at 151.13 32.512 0)
+		(at 151.13 33.02 0)
 		(effects
 			(font
@@
 	(bus
 		(pts
-			(xy 127 67.31) (xy 111.76 67.31)
-		)
-		(stroke
-			(width 0)
-			(type default)
-		)
-	)
-	(bus
-		(pts
-			(xy 120.65 110.49) (xy 120.65 73.66)
-		)
-		(stroke
-			(width 0)
-			(type default)
-		)
-	)
-	(bus
-		(pts
-			(xy 120.65 110.49) (xy 144.78 110.49)
-		)
-		(stroke
-			(width 0)
-			(type default)
-		)
-	)
-	(bus
-		(pts
-			(xy 127 104.14) (xy 127 67.31)
-		)
-		(stroke
-			(width 0)
-			(type default)
-		)
-	)
-	(bus
-		(pts
-			(xy 120.65 73.66) (xy 111.76 73.66)
-		)
-		(stroke
-			(width 0)
-			(type default)
-		)
-	)
-	(bus
-		(pts
-			(xy 127 104.14) (xy 144.78 104.14)
+			(xy 127 88.9) (xy 86.36 88.9)
+		)
+		(stroke
+			(width 0)
+			(type default)
+		)
+	)
+	(bus
+		(pts
+			(xy 120.65 132.08) (xy 120.65 95.25)
+		)
+		(stroke
+			(width 0)
+			(type default)
+		)
+	)
+	(bus
+		(pts
+			(xy 120.65 132.08) (xy 158.75 132.08)
+		)
+		(stroke
+			(width 0)
+			(type default)
+		)
+	)
+	(bus
+		(pts
+			(xy 127 125.73) (xy 127 88.9)
+		)
+		(stroke
+			(width 0)
+			(type default)
+		)
+	)
+	(bus
+		(pts
+			(xy 120.65 95.25) (xy 86.36 95.25)
+		)
+		(stroke
+			(width 0)
+			(type default)
+		)
+	)
+	(bus
+		(pts
+			(xy 127 125.73) (xy 158.75 125.73)
 		)
 		(stroke
@@
 	)
 	(sheet
-		(at 83.82 55.88)
+		(at 58.42 55.88)
 		(size 27.94 59.69)
 		(exclude_from_sim no)
@@
 		)
 		(property "Sheetname" "Right Keyboard Connector"
-			(at 83.82 55.1684 0)
+			(at 58.42 55.1684 0)
 			(effects
 				(font
@@
 		)
 		(property "Sheetfile" "right-conn.kicad_sch"
-			(at 83.82 116.1546 0)
+			(at 58.42 116.1546 0)
 			(effects
 				(font
@@
 		)
 		(pin "{COMMON_ROWS}" bidirectional
-			(at 111.76 67.31 0)
+			(at 86.36 88.9 0)
 			(effects
 				(font
@@
 		)
 		(pin "{RIGHT_COLUMNS}" bidirectional
-			(at 111.76 73.66 0)
+			(at 86.36 95.25 0)
 			(effects
 				(font
@@
 	)
 	(sheet
-		(at 144.78 92.71)
-		(size 64.77 43.18)
+		(at 158.75 75.565)
+		(size 43.18 26.035)
 		(exclude_from_sim no)
 		(in_bom yes)
@@
 			(color 0 0 0 0.0000)
 		)
+		(property "Sheetname" "GPIO Outputs"
+			(at 158.75 74.8534 0)
+			(effects
+				(font
+					(size 1.27 1.27)
+				)
+				(justify left bottom)
+			)
+		)
+		(property "Sheetfile" "gpio.kicad_sch"
+			(at 158.75 102.1846 0)
+			(effects
+				(font
+					(size 1.27 1.27)
+				)
+				(justify left top)
+			)
+		)
+		(instances
+			(project "69split"
+				(path "/d75b0717-10e3-4e20-afcb-05300684210e/4b966fee-8f5c-4a23-a90e-d8e6cc86345c"
+					(page "10")
+				)
+			)
+		)
+	)
+	(sheet
+		(at 158.75 114.3)
+		(size 43.18 31.75)
+		(exclude_from_sim no)
+		(in_bom yes)
+		(on_board yes)
+		(dnp no)
+		(fields_autoplaced yes)
+		(stroke
+			(width 0.1524)
+			(type solid)
+		)
+		(fill
+			(color 0 0 0 0.0000)
+		)
 		(property "Sheetname" "Right Matrix"
-			(at 144.78 91.9984 0)
+			(at 158.75 113.5884 0)
 			(effects
 				(font
@@
 		)
 		(property "Sheetfile" "right-matrix.kicad_sch"
-			(at 144.78 136.4746 0)
+			(at 158.75 145.9996 0)
 			(effects
 				(font
@@
 		)
 		(pin "{COMMON_ROWS}" input
-			(at 144.78 104.14 180)
+			(at 158.75 125.73 180)
 			(effects
 				(font
@@
 		)
 		(pin "{RIGHT_COLUMNS}" input
-			(at 144.78 110.49 180)
-			(effects
-				(font
+			(at 158.75 132.08 180)
+			(effects
+				(font

Commit message: I think schematic is done?
Other:
- sheet GPIO Outputs ports: added {GPIO_OUT}; removed none
- sheet Right Keyboard Connector ports: added {GPIO_OUT}; removed none
- title: Split Normal 69 -> 69SPLIT KEYBOARD
Changed lines of the file:
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@@
 	(paper "A4")
 	(title_block
-		(title "Split Normal 69")
+		(title "69SPLIT KEYBOARD")
 		(date "2025-06-11")
 	)
 	(rectangle
-		(start 73.66 62.865)
-		(end 228.6 149.225)
+		(start 73.66 74.295)
+		(end 234.95 142.24)
 		(stroke
 			(width 0)
@@
 	(bus
 		(pts
-			(xy 127 88.9) (xy 86.36 88.9)
-		)
-		(stroke
-			(width 0)
-			(type default)
-		)
-	)
-	(bus
-		(pts
-			(xy 120.65 132.08) (xy 120.65 95.25)
-		)
-		(stroke
-			(width 0)
-			(type default)
-		)
-	)
-	(bus
-		(pts
-			(xy 120.65 132.08) (xy 158.75 132.08)
-		)
-		(stroke
-			(width 0)
-			(type default)
-		)
-	)
-	(bus
-		(pts
-			(xy 127 125.73) (xy 127 88.9)
-		)
-		(stroke
-			(width 0)
-			(type default)
-		)
-	)
-	(bus
-		(pts
-			(xy 120.65 95.25) (xy 86.36 95.25)
-		)
-		(stroke
-			(width 0)
-			(type default)
-		)
-	)
-	(bus
-		(pts
-			(xy 127 125.73) (xy 158.75 125.73)
+			(xy 133.35 93.98) (xy 92.71 93.98)
+		)
+		(stroke
+			(width 0)
+			(type default)
+		)
+	)
+	(bus
+		(pts
+			(xy 127 121.92) (xy 127 100.33)
+		)
+		(stroke
+			(width 0)
+			(type default)
+		)
+	)
+	(bus
+		(pts
+			(xy 127 121.92) (xy 165.1 121.92)
+		)
+		(stroke
+			(width 0)
+			(type default)
+		)
+	)
+	(bus
+		(pts
+			(xy 92.71 81.28) (xy 165.1 81.28)
+		)
+		(stroke
+			(width 0)
+			(type default)
+		)
+	)
+	(bus
+		(pts
+			(xy 133.35 115.57) (xy 133.35 93.98)
+		)
+		(stroke
+			(width 0)
+			(type default)
+		)
+	)
+	(bus
+		(pts
+			(xy 127 100.33) (xy 92.71 100.33)
+		)
+		(stroke
+			(width 0)
+			(type default)
+		)
+	)
+	(bus
+		(pts
+			(xy 133.35 115.57) (xy 165.1 115.57)
 		)
 		(stroke
@@
 	)
 	(sheet
-		(at 58.42 55.88)
+		(at 64.77 67.31)
 		(size 27.94 59.69)
 		(exclude_from_sim no)
@@
 		)
 		(property "Sheetname" "Right Keyboard Connector"
-			(at 58.42 55.1684 0)
+			(at 64.77 66.5984 0)
 			(effects
 				(font
@@
 		)
 		(property "Sheetfile" "right-conn.kicad_sch"
-			(at 58.42 116.1546 0)
+			(at 64.77 127.5846 0)
 			(effects
 				(font
@@
 		)
 		(pin "{COMMON_ROWS}" bidirectional
-			(at 86.36 88.9 0)
+			(at 92.71 93.98 0)
 			(effects
 				(font
@@
 		)
 		(pin "{RIGHT_COLUMNS}" bidirectional
-			(at 86.36 95.25 0)
+			(at 92.71 100.33 0)
 			(effects
 				(font
 					(size 1.27 1.27)
 					(thickness 0.1588)
+				)
+				(justify right)
+			)
+		)
+		(pin "{GPIO_OUT}" input
+			(at 92.71 81.28 0)
+			(effects
+				(font
+					(size 1.27 1.27)
 				)
 				(justify right)
@@
 	)
 	(sheet
-		(at 158.75 75.565)
-		(size 43.18 26.035)
+		(at 165.1 67.31)
+		(size 43.18 21.59)
 		(exclude_from_sim no)
 		(in_bom yes)
@@
 		)
 		(property "Sheetname" "GPIO Outputs"
-			(at 158.75 74.8534 0)
+			(at 165.1 66.5984 0)
 			(effects
 				(font
@@
 		)
 		(property "Sheetfile" "gpio.kicad_sch"
-			(at 158.75 102.1846 0)
+			(at 165.1 89.4846 0)
 			(effects
 				(font
@@
 				)
 				(justify left top)
+			)
+		)
+		(pin "{GPIO_OUT}" input
+			(at 165.1 81.28 180)
+			(effects
+				(font
+					(size 1.27 1.27)
+				)
+				(justify left)
 			)
 		)
@@
 	)
 	(sheet
-		(at 158.75 114.3)
+		(at 165.1 104.14)
 		(size 43.18 31.75)
 		(exclude_from_sim no)
@@
 		)
 		(property "Sheetname" "Right Matrix"
-			(at 158.75 113.5884 0)
+			(at 165.1 103.4284 0)
 			(effects
 				(font
@@
 		)
 		(property "Sheetfile" "right-matrix.kicad_sch"
-			(at 158.75 145.9996 0)
+			(at 165.1 135.8396 0)
 			(effects
 				(font
@@
 		)
 		(pin "{COMMON_ROWS}" input
-			(at 158.75 125.73 180)
+			(at 165.1 115.57 180)
 			(effects
 				(font
@@
 		)
 		(pin "{RIGHT_COLUMNS}" input
-			(at 158.75 132.08 180)
-			(effects
-				(font
+			(at 165.1 121.92 180)
+			(effects
+				(font
