File: pcb/usb-conn.kicad_sch (KiCad schematic)
At the start: 6 parts, among them J1 USB_C_Receptacle_USB2.0_14P

Commit message: Added MPNs and footprints for I think everything.
Parts:
- C10: MPN (none) -> Generic; Rating (none) -> 10V
- J1: MPN DX07S016JA1R1500 -> DX07S016JA1R1500
- R2, R3: footprint Resistor_SMD:R_0805_2012Metric_Pad1.15x1.40mm_HandSolder -> Resistor_SMD:R_0603_1608Metric_Pad0.98x0.95mm_HandSolder; MPN (none) -> Generic
Changed lines of the file:
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@@
 			)
 		)
-		(property "Footprint" "Resistor_SMD:R_0805_2012Metric_Pad1.15x1.40mm_HandSolder"
+		(property "Footprint" "Resistor_SMD:R_0603_1608Metric_Pad0.98x0.95mm_HandSolder"
 			(at 127 90.932 90)
 			(effects
@@
 			)
 		)
+		(property "MPN" "Generic"
+			(at 127 92.71 90)
+			(effects
+				(font
+					(size 1.27 1.27)
+				)
+				(hide yes)
+			)
+		)
 		(pin "1"
 		)
@@
 			)
 		)
-		(property "Footprint" "Resistor_SMD:R_0805_2012Metric_Pad1.15x1.40mm_HandSolder"
+		(property "Footprint" "Resistor_SMD:R_0603_1608Metric_Pad0.98x0.95mm_HandSolder"
 			(at 127 96.012 90)
 			(effects
@@
 			)
 		)
+		(property "MPN" "Generic"
+			(at 127 97.79 90)
+			(effects
+				(font
+					(size 1.27 1.27)
+				)
+				(hide yes)
+			)
+		)
 		(pin "2"
 		)
@@
 			)
 		)
-		(property "MPN" "DX07S016JA1R1500"
+		(property "MPN" "DX07S016JA1R1500 "
 			(at 96.52 93.98 0)
 			(effects
@@
 		)
 		(property "Value" "GND"
-			(at 154.94 137.16 0)
-			(effects
-				(font
-					(size 1.27 1.27)
-				)
+			(at 157.48 133.3499 0)
+			(effects
+				(font
+					(size 1.27 1.27)
+				)
+				(justify right)
 			)
 		)
@@
 		(fields_autoplaced yes)
 		(property "Reference" "C10"
-			(at 171.45 80.0162 0)
+			(at 171.45 78.7462 0)
 			(effects
 				(font
@@
 		)
 		(property "Value" "10u"
-			(at 171.45 82.5562 0)
+			(at 171.45 81.2862 0)
 			(effects
 				(font
@@
 			)
 		)
+		(property "MPN" "Generic"
+			(at 168.91 81.28 0)
+			(effects
+				(font
+					(size 1.27 1.27)
+				)
+				(hide yes)
+			)
+		)
+		(property "Rating" "10V"
+			(at 171.45 83.8262 0)
+			(effects
+				(font
+					(size 1.27 1.27)
+				)
+				(justify left)
+			)
+		)

Commit message: Continuing...no one will read this but me.
Parts:
- C1: renamed from C10; footprint Capacitor_SMD:C_0805_2012Metric_Pad1.15x1.40mm_HandSolder -> Capacitor_SMD:C_0805_2012Metric_Pad1.18x1.45mm_HandSolder
- renumbered R2 to R1, R3 to R2, R7 to R3, R8 to R4
Other:
- note added: "USB CONNECTOR"
Changed lines of the file:
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@@
 		(members "VBUS" "D+" "D-")
+	)
+	(text "USB CONNECTOR"
+		(exclude_from_sim no)
+		(at 140.462 35.56 0)
+		(effects
+			(font
+				(face "Book Antiqua")
+				(size 7.62 7.62)
+				(color 0 0 0 1)
+			)
+		)
 	)
 	(junction
@@
 		(dnp no)
 		(fields_autoplaced yes)
-		(property "Reference" "#PWR0107"
+		(property "Reference" "#PWR03"
 			(at 88.9 125.73 0)
 			(effects
@@
 		(instances
 			(project "split-normal-69"
+				(path "/94301c1c-44b1-4926-ac38-8a25b84a2b23/619d845a-8c90-490b-ae7a-6c3e22416b6d/d3fe7daf-0d6e-41be-bc1c-53fc3114204a"
+					(reference "#PWR03")
+					(unit 1)
+				)
+			)
+			(project "69split"
 				(path "/d75b0717-10e3-4e20-afcb-05300684210e/a528eaf3-d99a-4f91-978f-500370d04b37/d3fe7daf-0d6e-41be-bc1c-53fc3114204a"
-					(reference "#PWR0107")
+					(reference "#PWR03")
 					(unit 1)
 				)
@@
 		(dnp no)
 		(fields_autoplaced yes)
-		(property "Reference" "R2"
+		(property "Reference" "R1"
 			(at 127 82.55 90)
 			(effects
@@
 		(instances
 			(project "split-normal-69"
+				(path "/94301c1c-44b1-4926-ac38-8a25b84a2b23/619d845a-8c90-490b-ae7a-6c3e22416b6d/d3fe7daf-0d6e-41be-bc1c-53fc3114204a"
+					(reference "R1")
+					(unit 1)
+				)
+			)
+			(project "69split"
 				(path "/d75b0717-10e3-4e20-afcb-05300684210e/a528eaf3-d99a-4f91-978f-500370d04b37/d3fe7daf-0d6e-41be-bc1c-53fc3114204a"
-					(reference "R2")
+					(reference "R1")
 					(unit 1)
 				)
@@
 		(dnp no)
 		(fields_autoplaced yes)
-		(property "Reference" "R3"
+		(property "Reference" "R2"
 			(at 127 101.6 90)
 			(effects
@@
 		(instances
 			(project "split-normal-69"
+				(path "/94301c1c-44b1-4926-ac38-8a25b84a2b23/619d845a-8c90-490b-ae7a-6c3e22416b6d/d3fe7daf-0d6e-41be-bc1c-53fc3114204a"
+					(reference "R2")
+					(unit 1)
+				)
+			)
+			(project "69split"
 				(path "/d75b0717-10e3-4e20-afcb-05300684210e/a528eaf3-d99a-4f91-978f-500370d04b37/d3fe7daf-0d6e-41be-bc1c-53fc3114204a"
-					(reference "R3")
+					(reference "R2")
 					(unit 1)
 				)
@@
 		(dnp no)
 		(fields_autoplaced yes)
-		(property "Reference" "#PWR0117"
+		(property "Reference" "#PWR01"
 			(at 125.73 78.74 0)
 			(effects
@@
 		(instances
 			(project "split-normal-69"
+				(path "/94301c1c-44b1-4926-ac38-8a25b84a2b23/619d845a-8c90-490b-ae7a-6c3e22416b6d/d3fe7daf-0d6e-41be-bc1c-53fc3114204a"
+					(reference "#PWR01")
+					(unit 1)
+				)
+			)
+			(project "69split"
 				(path "/d75b0717-10e3-4e20-afcb-05300684210e/a528eaf3-d99a-4f91-978f-500370d04b37/d3fe7daf-0d6e-41be-bc1c-53fc3114204a"
-					(reference "#PWR0117")
+					(reference "#PWR01")
 					(unit 1)
 				)
@@
 		(instances
 			(project "split-normal-69"
+				(path "/94301c1c-44b1-4926-ac38-8a25b84a2b23/619d845a-8c90-490b-ae7a-6c3e22416b6d/d3fe7daf-0d6e-41be-bc1c-53fc3114204a"
+					(reference "J1")
+					(unit 1)
+				)
+			)
+			(project "69split"
 				(path "/d75b0717-10e3-4e20-afcb-05300684210e/a528eaf3-d99a-4f91-978f-500370d04b37/d3fe7daf-0d6e-41be-bc1c-53fc3114204a"
 					(reference "J1")
@@
 		(dnp no)
 		(fields_autoplaced yes)
-		(property "Reference" "#PWR05"
+		(property "Reference" "#PWR02"
 			(at 168.91 90.17 0)
 			(effects
@@
 		(instances
 			(project "split-normal-69"
+				(path "/94301c1c-44b1-4926-ac38-8a25b84a2b23/619d845a-8c90-490b-ae7a-6c3e22416b6d/d3fe7daf-0d6e-41be-bc1c-53fc3114204a"
+					(reference "#PWR02")
+					(unit 1)
+				)
+			)
+			(project "69split"
 				(path "/d75b0717-10e3-4e20-afcb-05300684210e/a528eaf3-d99a-4f91-978f-500370d04b37/d3fe7daf-0d6e-41be-bc1c-53fc3114204a"
-					(reference "#PWR05")
+					(reference "#PWR02")
 					(unit 1)
 				)
@@
 		(dnp no)
 		(fields_autoplaced yes)
-		(property "Reference" "R8"
+		(property "Reference" "R4"
 			(at 160.02 107.9499 0)
 			(effects
@@
 		(instances
 			(project "split-normal-69"
+				(path "/94301c1c-44b1-4926-ac38-8a25b84a2b23/619d845a-8c90-490b-ae7a-6c3e22416b6d/d3fe7daf-0d6e-41be-bc1c-53fc3114204a"
+					(reference "R4")
+					(unit 1)
+				)
+			)
+			(project "69split"
 				(path "/d75b0717-10e3-4e20-afcb-05300684210e/a528eaf3-d99a-4f91-978f-500370d04b37/d3fe7daf-0d6e-41be-bc1c-53fc3114204a"
-					(reference "R8")
+					(reference "R4")
 					(unit 1)
 				)
@@
 		(instances
 			(project "split-normal-69"
+				(path "/94301c1c-44b1-4926-ac38-8a25b84a2b23/619d845a-8c90-490b-ae7a-6c3e22416b6d/d3fe7daf-0d6e-41be-bc1c-53fc3114204a"
+					(reference "#PWR04")
+					(unit 1)
+				)
+			)
+			(project "69split"
 				(path "/d75b0717-10e3-4e20-afcb-05300684210e/a528eaf3-d99a-4f91-978f-500370d04b37/d3fe7daf-0d6e-41be-bc1c-53fc3114204a"
 					(reference "#PWR04")
@@
 		(dnp no)
 		(fields_autoplaced yes)
-		(property "Reference" "R7"
+		(property "Reference" "R3"
 			(at 149.86 102.8699 0)
 			(effects
@@
 		(instances
 			(project "split-normal-69"
+				(path "/94301c1c-44b1-4926-ac38-8a25b84a2b23/619d845a-8c90-490b-ae7a-6c3e22416b6d/d3fe7daf-0d6e-41be-bc1c-53fc3114204a"
+					(reference "R3")
+					(unit 1)
+				)
+			)
+			(project "69split"
 				(path "/d75b0717-10e3-4e20-afcb-05300684210e/a528eaf3-d99a-4f91-978f-500370d04b37/d3fe7daf-0d6e-41be-bc1c-53fc3114204a"
-					(reference "R7")
+					(reference "R3")
 					(unit 1)
 				)
@@
 		(dnp no)
 		(fields_autoplaced yes)
-		(property "Reference" "C10"
+		(property "Reference" "C1"
 			(at 171.45 78.7462 0)
 			(effects
@@
 			)
 		)
-		(property "Footprint" "Capacitor_SMD:C_0805_2012Metric_Pad1.15x1.40mm_HandSolder"
+		(property "Footprint" "Capacitor_SMD:C_0805_2012Metric_Pad1.18x1.45mm_HandSolder"
 			(at 168.91 81.28 0)
 			(effects
@@
 		(instances
 			(project "split-normal-69"
+				(path "/94301c1c-44b1-4926-ac38-8a25b84a2b23/619d845a-8c90-490b-ae7a-6c3e22416b6d/d3fe7daf-0d6e-41be-bc1c-53fc3114204a"
+					(reference "C1")
+					(unit 1)
+				)
+			)
+			(project "69split"
 				(path "/d75b0717-10e3-4e20-afcb-05300684210e/a528eaf3-d99a-4f91-978f-500370d04b37/d3fe7daf-0d6e-41be-bc1c-53fc3114204a"
-					(reference "C10")
-					(unit 1)
-				)
+					(reference "C1")
+					(unit 1)
+				)

Commit message: I think schematic is done?
Other:
- title: Split Normal 69 -> 69SPLIT KEYBOARD
Changed lines of the file:
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@@
 	(paper "A4")
 	(title_block
-		(title "Split Normal 69")
+		(title "69SPLIT KEYBOARD")
 		(date "2025-06-11")
 	)
