File: pcb/69split-left/atmega32u4.kicad_sch (KiCad schematic)
At the start: 16 parts, among them J2 Conn_02x03_Odd_Even, SW1 SW_Push, U1 ATmega32U4-AU, Y1 Crystal

Commit message: Final touches.
Parts:
- C6: value 1u -> 100n
- Y1: MPN ABL-16.000MHz-B4Y -> ABL-8.000MHZ-B4Y-T; Rating 16 MHz -> 8 MHz
Other:
- note removed: "GPIOs: 330R on right side for 10mA limit @ 3V3 and 15mA @ 5V"
- note removed: "Route D+/- as differential pairs."
- moved on the sheet: J2
