File: pcb/69split-left/usb-conn.kicad_sch (KiCad schematic)
At the start: 8 parts, among them J1 USB_C_Receptacle_USB2.0_16P, U3 TPD2E2U06DCK

Commit message: Final touches.
Parts:
- R3, R4: MPN MCT06030C5101FPW00 -> Generic
Changed lines of the file:
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@@
 	(text "Route D+/- as differential pairs.\nPlace resistors close to connector.\nFor 90 Ohm impedance coplanar differential pairs,\nWidth: 16 mil (~0.4 mm)\nClearance: 5 mil (~0.12 mm)\n\nSource\nhttps://resources.altium.com/p/routing-requirements-usb-20-2-layer-pcb"
 		(exclude_from_sim no)
-		(at 206.502 114.808 0)
+		(at 201.422 118.11 0)
 		(effects
 			(font
@@
 	)
 	(hierarchical_label "USB_5V"
-		(shape input)
+		(shape output)
 		(at 259.08 78.74 0)
 		(effects
@@
 			)
 		)
-		(property "Untitled Field" ""
-			(at 125.73 92.71 90)
-			(effects
-				(font
-					(size 1.27 1.27)
-				)
-				(hide yes)
-			)
-		)
 		(pin "1"
 		)
@@
 			)
 		)
-		(property "Untitled Field" ""
-			(at 125.73 97.79 90)
-			(effects
-				(font
-					(size 1.27 1.27)
-				)
-				(hide yes)
-			)
-		)
 		(pin "2"
 		)
@@
 			)
 		)
-		(property "Untitled Field" ""
-			(at 96.52 93.98 0)
-			(effects
-				(font
-					(size 1.27 1.27)
-				)
-				(hide yes)
-			)
-		)
 		(pin "B1"
 		)
@@
 			)
 		)
-		(property "MPN" "MCT06030C5101FPW00"
+		(property "MPN" "Generic"
 			(at 176.53 110.49 0)
 			(effects
@@
 		)
 		(property "Key" ""
-			(at 176.53 110.49 0)
-			(effects
-				(font
-					(size 1.27 1.27)
-				)
-				(hide yes)
-			)
-		)
-		(property "Untitled Field" ""
 			(at 176.53 110.49 0)
 			(effects
@@
 			)
 		)
-		(property "MPN" "MCT06030C5101FPW00"
+		(property "MPN" "Generic"
 			(at 171.45 105.41 0)
 			(effects
@@
 		)
 		(property "Key" ""
-			(at 171.45 105.41 0)
-			(effects
-				(font
-					(size 1.27 1.27)
-				)
-				(hide yes)
-			)
-		)
-		(property "Untitled Field" ""
 			(at 171.45 105.41 0)
 			(effects
@@
 			(at 204.47 81.28 0)
 			(effects
-				(font
-					(size 1.27 1.27)
-				)
-				(hide yes)
-			)
-		)
-		(property "Untitled Field" ""
-			(at 204.47 81.28 0)
-			(effects
