File: pcb/69split-right/69split-right.kicad_sch (KiCad schematic)
At the start: 0 parts

Commit message: Final touches.
Other:
- note added: "L + R 42mA + 76mA @ 5V 25mA + 51mA @ 3V3 Typical current draw when everythin is in use except the breakout header."
Changed lines of the file:
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@@
 		(title "69SPLIT")
 		(date "2025-07-28")
-		(rev "1")
+		(rev "A")
 		(company "Yiannis Michael")
 		(comment 1 "Yiannis Michael")
@@
 	)
 	(rectangle
-		(start 143.51 81.915)
-		(end 220.98 149.86)
+		(start 146.05 92.075)
+		(end 223.52 160.02)
 		(stroke
 			(width 0)
@@
 	)
 	(arc
-		(start 95.885 76.2)
-		(mid 115.57 64.2281)
-		(end 135.255 76.2)
+		(start 98.425 86.36)
+		(mid 118.11 74.3881)
+		(end 137.795 86.36)
 		(stroke
 			(width 0)
@@
 	)
 	(rectangle
-		(start 60.96 76.2)
-		(end 112.395 130.81)
+		(start 63.5 86.36)
+		(end 114.935 140.97)
 		(stroke
 			(width 0)
@@
 		)
 	)
+	(text "L + R\n42mA + 76mA @ 5V\n25mA + 51mA @ 3V3\n\nTypical current draw when everythin is in use\nexcept the breakout header."
+		(exclude_from_sim no)
+		(at 210.566 30.48 0)
+		(effects
+			(font
+				(size 2 2)
+			)
+			(justify left)
+		)
+	)
 	(text "GPIO Outputs"
 		(exclude_from_sim no)
-		(at 205.74 50.8 0)
+		(at 208.28 60.96 0)
 		(effects
 			(font
@@
 	(text "Keyboard USB-C Connection"
 		(exclude_from_sim no)
-		(at 101.6 60.96 0)
+		(at 104.14 71.12 0)
 		(effects
 			(font
@@
 	(text "USB-C to PC"
 		(exclude_from_sim no)
-		(at 63.5 50.8 0)
+		(at 66.04 60.96 0)
 		(effects
 			(font
@@
 	(text "Left Keyboard"
 		(exclude_from_sim no)
-		(at 86.36 101.6 0)
+		(at 88.9 111.76 0)
 		(effects
 			(font
@@
 	(bus
 		(pts
-			(xy 180.34 121.92) (xy 180.34 93.98)
+			(xy 182.88 132.08) (xy 182.88 104.14)
 		)
 		(stroke
@@
 	(polyline
 		(pts
-			(xy 215.9 53.34) (xy 215.9 76.2)
+			(xy 218.44 63.5) (xy 218.44 86.36)
 		)
 		(stroke
@@
 	(polyline
 		(pts
-			(xy 71.12 53.34) (xy 71.12 76.2)
+			(xy 73.66 63.5) (xy 73.66 86.36)
 		)
 		(stroke
@@
 	(bus
 		(pts
-			(xy 190.5 93.98) (xy 185.42 93.98)
+			(xy 193.04 104.14) (xy 187.96 104.14)
 		)
 		(stroke
@@
 	(polyline
 		(pts
-			(xy 210.82 53.34) (xy 210.82 76.2)
+			(xy 213.36 63.5) (xy 213.36 86.36)
 		)
 		(stroke
@@
 	(bus
 		(pts
-			(xy 185.42 128.27) (xy 175.26 128.27)
-		)
-		(stroke
-			(width 0)
-			(type default)
-		)
-	)
-	(bus
-		(pts
-			(xy 180.34 93.98) (xy 162.56 93.98)
-		)
-		(stroke
-			(width 0)
-			(type default)
-		)
-	)
-	(bus
-		(pts
-			(xy 175.26 134.62) (xy 190.5 134.62)
-		)
-		(stroke
-			(width 0)
-			(type default)
-		)
-	)
-	(bus
-		(pts
-			(xy 162.56 86.36) (xy 190.5 86.36)
+			(xy 187.96 138.43) (xy 177.8 138.43)
+		)
+		(stroke
+			(width 0)
+			(type default)
+		)
+	)
+	(bus
+		(pts
+			(xy 182.88 104.14) (xy 165.1 104.14)
+		)
+		(stroke
+			(width 0)
+			(type default)
+		)
+	)
+	(bus
+		(pts
+			(xy 177.8 144.78) (xy 193.04 144.78)
+		)
+		(stroke
+			(width 0)
+			(type default)
+		)
+	)
+	(bus
+		(pts
+			(xy 165.1 96.52) (xy 193.04 96.52)
 		)
 		(stroke
@@
 	(polyline
 		(pts
-			(xy 66.04 53.34) (xy 66.04 76.2)
+			(xy 68.58 63.5) (xy 68.58 86.36)
 		)
 		(stroke
@@
 	(bus
 		(pts
-			(xy 175.26 121.92) (xy 180.34 121.92)
-		)
-		(stroke
-			(width 0)
-			(type default)
-		)
-	)
-	(bus
-		(pts
-			(xy 185.42 93.98) (xy 185.42 128.27)
+			(xy 177.8 132.08) (xy 182.88 132.08)
+		)
+		(stroke
+			(width 0)
+			(type default)
+		)
+	)
+	(bus
+		(pts
+			(xy 187.96 104.14) (xy 187.96 138.43)
 		)
 		(stroke
@@
 	)
 	(sheet
-		(at 190.5 121.92)
+		(at 193.04 132.08)
 		(size 27.94 17.78)
 		(exclude_from_sim no)
@@
 		)
 		(property "Sheetname" "Right Matrix"
-			(at 190.5 121.2084 0)
+			(at 193.04 131.3684 0)
 			(effects
 				(font
@@
 		)
 		(property "Sheetfile" "right-matrix.kicad_sch"
-			(at 190.5 140.2846 0)
+			(at 193.04 150.4446 0)
 			(effects
 				(font
@@
 			)
 		)
-		(pin "{RIGHT_MATRIX}" input
-			(at 190.5 134.62 180)
+		(pin "{RIGHT_MATRIX}" bidirectional
+			(at 193.04 144.78 180)
 			(effects
 				(font
@@
 	)
 	(sheet
-		(at 152.4 116.84)
+		(at 154.94 127)
 		(size 22.86 22.86)
 		(exclude_from_sim no)
@@
 		)
 		(property "Sheetname" "IO Expander"
-			(at 152.4 116.1284 0)
+			(at 154.94 126.2884 0)
 			(effects
 				(font
@@
 		)
 		(property "Sheetfile" "io-expander.kicad_sch"
-			(at 152.4 140.2846 0)
+			(at 154.94 150.4446 0)
 			(effects
 				(font
@@
 			)
 		)
-		(pin "{I2C}" input
-			(at 175.26 121.92 0)
+		(pin "{I2C}" bidirectional
+			(at 177.8 132.08 0)
 			(effects
 				(font
@@
 			)
 		)
-		(pin "{RIGHT_MATRIX}" input
-			(at 175.26 134.62 0)
+		(pin "{RIGHT_MATRIX}" bidirectional
+			(at 177.8 144.78 0)
 			(effects
 				(font
@@
 			)
 		)
-		(pin "{GPIO_EXP_OUT}" input
-			(at 175.26 128.27 0)
+		(pin "{GPIO_EXP_OUT}" bidirectional
+			(at 177.8 138.43 0)
 			(effects
 				(font
@@
 	)
 	(sheet
-		(at 132.08 76.2)
+		(at 134.62 86.36)
 		(size 30.48 25.4)
 		(exclude_from_sim no)
@@
 		)
 		(property "Sheetname" "Right Keyboard Connector"
-			(at 137.795 75.692 0)
+			(at 140.335 85.852 0)
 			(effects
 				(font
@@
 		)
 		(property "Sheetfile" "right-conn.kicad_sch"
-			(at 132.715 102.362 0)
+			(at 135.255 112.522 0)
 			(effects
 				(font
@@
 			)
 		)
-		(pin "{GPIO_OUT}" input
-			(at 162.56 86.36 0)
+		(pin "{GPIO_OUT}" output
+			(at 165.1 96.52 0)
 			(effects
 				(font
@@
 			)
 		)
-		(pin "{I2C}" input
-			(at 162.56 93.98 0)
+		(pin "{I2C}" bidirectional
+			(at 165.1 104.14 0)
 			(effects
 				(font
@@
 	)
 	(sheet
-		(at 190.5 76.2)
+		(at 193.04 86.36)
 		(size 33.02 25.4)
 		(exclude_from_sim no)
@@
 		)
 		(property "Sheetname" "GPIO Outputs"
-			(at 190.5 75.4884 0)
+			(at 193.04 85.6484 0)
 			(effects
 				(font
@@
 		)
 		(property "Sheetfile" "gpio.kicad_sch"
-			(at 190.5 102.1846 0)
+			(at 193.04 112.3446 0)
 			(effects
 				(font
@@
 		)
 		(pin "{GPIO_OUT}" input
-			(at 190.5 86.36 180)
+			(at 193.04 96.52 180)
 			(effects
 				(font
@@
 			)
 		)
-		(pin "{GPIO_EXP_OUT}" input
-			(at 190.5 93.98 180)
-			(effects
-				(font
+		(pin "{GPIO_EXP_OUT}" bidirectional
+			(at 193.04 104.14 180)
+			(effects
+				(font
