File: pcb/69split-right/69split-right.kicad_sch (KiCad schematic)
At the start: 0 parts

Commit message: More final touches fml.
Other:
- sheet GPIO Outputs: file gpio.kicad_sch -> 69split-right-sheets/gpio.kicad_sch
- sheet IO Expander: file io-expander.kicad_sch -> 69split-right-sheets/io-expander.kicad_sch
- sheet Right Keyboard Connector: file right-conn.kicad_sch -> 69split-right-sheets/right-conn.kicad_sch
- sheet Right Matrix: file right-matrix.kicad_sch -> 69split-right-sheets/right-matrix.kicad_sch
Changed lines of the file:
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@@
 			)
 		)
-		(property "Sheetfile" "right-matrix.kicad_sch"
+		(property "Sheetfile" "69split-right-sheets/right-matrix.kicad_sch"
 			(at 193.04 150.4446 0)
 			(effects
@@
 		(on_board yes)
 		(dnp no)
-		(fields_autoplaced yes)
 		(stroke
 			(width 0.1524)
@@
 			)
 		)
-		(property "Sheetfile" "io-expander.kicad_sch"
-			(at 154.94 150.4446 0)
+		(property "Sheetfile" "69split-right-sheets/io-expander.kicad_sch"
+			(at 129.794 150.368 0)
 			(effects
 				(font
@@
 			)
 		)
-		(property "Sheetfile" "right-conn.kicad_sch"
+		(property "Sheetfile" "69split-right-sheets/right-conn.kicad_sch"
 			(at 135.255 112.522 0)
 			(effects
@@
 			)
 		)
-		(property "Sheetfile" "gpio.kicad_sch"
+		(property "Sheetfile" "69split-right-sheets/gpio.kicad_sch"
 			(at 193.04 112.3446 0)
 			(effects
