File: pcb/69split-right/69split-right.kicad_pcb (KiCad board)
At the start: 2 copper layers, 186.1 x 108.9 mm, 91 parts, among them J1 Conn_01x03_Socket, J2 USB_C_Receptacle_USB2.0_16P, J3 Conn_01x03_Socket, SW1 SW_Push, SW10 SW_Push, SW11 SW_Push, SW12 SW_Push, SW13 SW_Push, SW14 SW_Push, SW15 SW_Push, SW16 SW_Push, SW17 SW_Push, SW18 SW_Push, SW19 SW_Push, SW2 SW_Push, SW20 SW_Push, SW21 SW_Push, SW22 SW_Push, SW23 SW_Push, SW24 SW_Push, SW25 SW_Push, SW26 SW_Push, SW27 SW_Push, SW28 SW_Push, SW29 SW_Push, SW3 SW_Push, SW30 SW_Push, SW31 SW_Push, SW32 SW_Push, SW33 SW_Push, SW34 SW_Push, SW35 SW_Push, SW36 SW_Push, SW37 SW_Push, SW38 SW_Push, SW39 SW_Push, SW4 SW_Push, SW5 SW_Push, SW6 SW_Push, SW7 SW_Push, SW8 SW_Push, SW9 SW_Push, U1 MCP23017_SS

Commit message: Added and updated READMEs and some other minor changes.
Routing:
- net VCC: track 190.9 -> 194.0 mm, vias 6 -> 12
Changed lines of the file:
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@@
 	(segment
 		(start 81.21 44.99)
-		(end 90.387355 44.99)
+		(end 88.87 44.99)
 		(width 0.4)
 		(layer "F.Cu")
@@
 	)
 	(segment
+		(start 90.36 44.99)
+		(end 90.387355 44.99)
+		(width 0.4)
+		(layer "F.Cu")
+		(net 45)
+	)
+	(segment
 		(start 220.52 60.44)
 		(end 220.52 61.2925)
@@
 	)
 	(segment
-		(start 224.29 67.0625)
-		(end 224.4225 66.93)
-		(width 0.2)
+		(start 210.865 44.305)
+		(end 210.85 44.29)
+		(width 0.4)
 		(layer "F.Cu")
 		(net 45)
 	)
 	(segment
-		(start 90.387355 44.99)
-		(end 91.087355 44.29)
-		(width 0.4)
+		(start 224.29 67.0625)
+		(end 224.4225 66.93)
+		(width 0.2)
 		(layer "F.Cu")
 		(net 45)
@@
 	)
 	(segment
+		(start 212.385 44.305)
+		(end 216.53 48.45)
+		(width 0.4)
+		(layer "F.Cu")
+		(net 45)
+	)
+	(segment
 		(start 233.42 67.87)
 		(end 233.42 64.9025)
@@
 	)
 	(segment
-		(start 91.087355 44.29)
-		(end 212.37 44.29)
+		(start 212.385 44.305)
+		(end 210.865 44.305)
 		(width 0.4)
 		(layer "F.Cu")
@@
 	)
 	(segment
+		(start 88.87 44.99)
+		(end 89.63 44.99)
+		(width 0.4)
+		(layer "F.Cu")
+		(net 45)
+	)
+	(segment
 		(start 216.53 59.66)
 		(end 217.06 60.19)
@@
 	(segment
 		(start 212.37 44.29)
-		(end 216.53 48.45)
+		(end 212.385 44.305)
 		(width 0.4)
 		(layer "F.Cu")
@@
 	)
 	(segment
+		(start 89.63 44.99)
+		(end 90.36 44.99)
+		(width 0.4)
+		(layer "F.Cu")
+		(net 45)
+	)
+	(segment
 		(start 220.34 67.95)
 		(end 220.005 67.95)
@@
 	)
 	(via
+		(at 212.385 44.305)
+		(size 0.6)
+		(drill 0.3)
+		(layers "F.Cu" "B.Cu")
+		(net 45)
+	)
+	(via
 		(at 227.88 67.93)
 		(size 0.6)
@@
 	)
 	(via
+		(at 90.36 44.99)
+		(size 0.6)
+		(drill 0.3)
+		(layers "F.Cu" "B.Cu")
+		(net 45)
+	)
+	(via
 		(at 227.88 61.74)
 		(size 0.6)
@@
 		(net 45)
 	)
+	(via
+		(at 210.85 44.29)
+		(size 0.6)
+		(drill 0.3)
+		(layers "F.Cu" "B.Cu")
+		(net 45)
+	)
+	(via
+		(at 211.64 44.29)
+		(size 0.6)
+		(drill 0.3)
+		(layers "F.Cu" "B.Cu")
+		(net 45)
+	)
+	(via
+		(at 88.87 44.99)
+		(size 0.6)
+		(drill 0.3)
+		(layers "F.Cu" "B.Cu")
+		(net 45)
+	)
+	(via
+		(at 89.63 44.99)
+		(size 0.6)
+		(drill 0.3)
+		(layers "F.Cu" "B.Cu")
+		(net 45)
+	)
 	(segment
 		(start 233.339265 67.950735)
@@
 	)
 	(segment
+		(start 90.36 44.99)
+		(end 88.87 44.99)
+		(width 0.4)
+		(layer "B.Cu")
+		(net 45)
+	)
+	(segment
 		(start 227.58 61.44)
 		(end 224.87 61.44)
@@
 	)
 	(segment
+		(start 210.85 44.29)
+		(end 211.64 44.29)
+		(width 0.4)
+		(layer "B.Cu")
+		(net 45)
+	)
+	(segment
+		(start 90.36 44.99)
+		(end 91.06 44.29)
+		(width 0.4)
+		(layer "B.Cu")
+		(net 45)
+	)
+	(segment
+		(start 91.06 44.29)
+		(end 210.85 44.29)
+		(width 0.4)
+		(layer "B.Cu")
+		(net 45)
+	)
+	(segment
+		(start 211.64 44.29)
+		(end 212.37 44.29)
+		(width 0.4)
+		(layer "B.Cu")
+		(net 45)
+	)
+	(segment
 		(start 225.089138 56.096508)
 		(end 225.085646 56.1)
@@
 	)
 	(segment
-		(start 80.715 125.84)
-		(end 80.715 127.32875)
+		(start 235.29 60.97)
+		(end 235.271 60.989)
 		(width 0.2)
 		(layer "F.Cu")
@@
 	)
 	(segment
-		(start 235.29 60.97)
-		(end 235.271 60.989)
+		(start 76.377355 53.934855)
+		(end 75.9525 53.51)
 		(width 0.2)
 		(layer "F.Cu")
@@
 	)
 	(segment
-		(start 76.377355 53.934855)
-		(end 75.9525 53.51)
+		(start 81.12 127.73375)
+		(end 83.09625 129.71)
 		(width 0.2)
 		(layer "F.Cu")
@@
 	)
 	(segment
-		(start 80.715 110.66)
-		(end 80.715 125.84)
+		(start 232.445 60.835)
+		(end 232.46 60.82)
 		(width 0.2)
 		(layer "F.Cu")
@@
 	)
 	(segment
-		(start 232.445 60.835)
-		(end 232.46 60.82)
+		(start 81.1 125.83)
+		(end 81.1 111.045)
+		(width 0.2)
+		(layer "F.Cu")
+		(net 52)
+	)
+	(segment
+		(start 81.1 125.83)
+		(end 81.12 125.85)
 		(width 0.2)
 		(layer "F.Cu")
@@
 	)
 	(segment
-		(start 80.715 127.32875)
-		(end 83.09625 129.71)
+		(start 81.12 125.85)
+		(end 81.12 127.73375)
 		(width 0.2)
 		(layer "F.Cu")
@@
 	)
 	(segment
+		(start 81.1 111.045)
+		(end 80.715 110.66)
+		(width 0.2)
+		(layer "F.Cu")
+		(net 52)
+	)
+	(segment
 		(start 71.74 110.54)
 		(end 71.74 92.16)
@@
 	)
 	(via
-		(at 80.715 125.84)
+		(at 81.1 125.83)
 		(size 0.6)
 		(drill 0.3)
@@
 	)
 	(segment
-		(start 80.725 125.83)
-		(end 80.715 125.84)
+		(start 81.1 125.83)
+		(end 235.41 125.83)
 		(width 0.2)
 		(layer "B.Cu")
@@
 	)
 	(segment
-		(start 235.41 125.83)
-		(end 80.725 125.83)
-		(width 0.2)
-		(layer "B.Cu")
-		(net 52)
-	)
-	(segment
 		(start 71.86 110.66)
 		(end 80.715 110.66)
@@
 	)
 	(segment
-		(start 90.24 91.61)
-		(end 89.5 91.61)
-		(width 0.2)
-		(layer "F.Cu")
-		(net 53)
-	)
-	(segment
 		(start 95.657355 72.49)
 		(end 95.657355 54.164855)
@@
 	)
 	(segment
+		(start 86.04 88.15)
+		(end 86.04 73.1225)
+		(width 0.2)
+		(layer "F.Cu")
+		(net 53)
+	)
+	(segment
+		(start 89.5 91.61)
+		(end 86.04 88.15)
+		(width 0.2)
+		(layer "F.Cu")
+		(net 53)
+	)
+	(segment
 		(start 90.977355 110.66)
 		(end 90.947355 110.63)
@@
 	)
 	(segment
-		(start 85.4775 87.5875)
+		(start 86.04 73.1225)
 		(end 85.4775 72.56)
 		(width 0.2)
@@
 	)
 	(segment
+		(start 90.24 91.61)
+		(end 89.5 91.61)
+		(width 0.2)
+		(layer "F.Cu")
+		(net 53)
+	)
+	(segment
 		(start 236.491 60.21)
 		(end 236.611 60.33)
@@
 	)
 	(segment
-		(start 89.5 91.61)
-		(end 85.4775 87.5875)
-		(width 0.2)
-		(layer "F.Cu")
-		(net 53)
-	)
-	(segment
 		(start 232.905 60.185)
 		(end 233.01 60.08)
@@
 		(filled_areas_thickness no)
 		(fill yes
-			(thermal_gap 0.5)
+			(thermal_gap 0.2)
 			(thermal_bridge_width 0.5)
 		)

Commit message: Ordered the PCBs and parts!
Routing:
- net /IO Expander/COL8: track 271.3 -> 270.3 mm
- net /IO Expander/COL11: track 229.3 -> 228.5 mm
- net GND: vias 28 -> 29
Other:
- outline, holes or cut-outs redrawn

Commit message: Fix column number labels
Before it started from COL6 but it should start from COL7 because COL6
is on the left PCB.
Connections:
- SW1 pad 1: /IO Expander/COL6 -> /IO Expander/COL7
- SW10 pad 1: /IO Expander/COL7 -> /IO Expander/COL8
- SW11 pad 1: /IO Expander/COL8 -> /IO Expander/COL9
- SW12 pad 1: /IO Expander/COL9 -> /IO Expander/COL10
- SW13 pad 1: /IO Expander/COL10 -> /IO Expander/COL11
- SW14 pad 1: /IO Expander/COL11 -> /IO Expander/COL12
- SW15 pad 1: /IO Expander/COL12 -> /IO Expander/COL13
- SW16 pad 1: /IO Expander/COL13 -> /IO Expander/COL14
- SW17 pad 1: /IO Expander/COL6 -> /IO Expander/COL7
- SW18 pad 1: /IO Expander/COL7 -> /IO Expander/COL8
- SW19 pad 1: /IO Expander/COL8 -> /IO Expander/COL9
- SW2 pad 1: /IO Expander/COL7 -> /IO Expander/COL8
- SW20 pad 1: /IO Expander/COL9 -> /IO Expander/COL10
- SW21 pad 1: /IO Expander/COL10 -> /IO Expander/COL11
- SW22 pad 1: /IO Expander/COL11 -> /IO Expander/COL12
- SW23 pad 1: /IO Expander/COL12 -> /IO Expander/COL13
- SW24 pad 1: /IO Expander/COL13 -> /IO Expander/COL14
- SW25 pad 1: /IO Expander/COL6 -> /IO Expander/COL7
- SW26 pad 1: /IO Expander/COL7 -> /IO Expander/COL8
- SW27 pad 1: /IO Expander/COL8 -> /IO Expander/COL9
- SW28 pad 1: /IO Expander/COL9 -> /IO Expander/COL10
- SW29 pad 1: /IO Expander/COL10 -> /IO Expander/COL11
- SW3 pad 1: /IO Expander/COL8 -> /IO Expander/COL9
- SW30 pad 1: /IO Expander/COL11 -> /IO Expander/COL12
- SW31 pad 1: /IO Expander/COL12 -> /IO Expander/COL13
- SW32 pad 1: /IO Expander/COL13 -> /IO Expander/COL14
- SW33 pad 1: /IO Expander/COL6 -> /IO Expander/COL7
- SW34 pad 1: /IO Expander/COL8 -> /IO Expander/COL9
- SW35 pad 1: /IO Expander/COL9 -> /IO Expander/COL10
- SW36 pad 1: /IO Expander/COL10 -> /IO Expander/COL11
- SW37 pad 1: /IO Expander/COL11 -> /IO Expander/COL12
- SW38 pad 1: /IO Expander/COL12 -> /IO Expander/COL13
- SW39 pad 1: /IO Expander/COL13 -> /IO Expander/COL14
- SW4 pad 1: /IO Expander/COL9 -> /IO Expander/COL10
- SW5 pad 1: /IO Expander/COL10 -> /IO Expander/COL11
- SW6 pad 1: /IO Expander/COL11 -> /IO Expander/COL12
- SW7 pad 1: /IO Expander/COL12 -> /IO Expander/COL13
- SW8 pad 1: /IO Expander/COL13 -> /IO Expander/COL14
- SW9 pad 1: /IO Expander/COL6 -> /IO Expander/COL7
- U1 pad 21: /IO Expander/COL6 -> /IO Expander/COL7
- U1 pad 22: /IO Expander/COL7 -> /IO Expander/COL8
- U1 pad 23: /IO Expander/COL8 -> /IO Expander/COL9
- U1 pad 24: /IO Expander/COL9 -> /IO Expander/COL10
- U1 pad 25: /IO Expander/COL10 -> /IO Expander/COL11
- U1 pad 26: /IO Expander/COL11 -> /IO Expander/COL12
- U1 pad 27: /IO Expander/COL12 -> /IO Expander/COL13
- U1 pad 28: /IO Expander/COL13 -> /IO Expander/COL14
Routing:
- net /IO Expander/COL6: track 322.7 -> 0.00 mm, vias 6 -> 0
- net /IO Expander/COL14: track 0.00 -> 109.0 mm, vias 0 -> 4
- net /IO Expander/COL13: track 109.0 -> 178.7 mm, vias 4 -> 5
- net /IO Expander/COL12: track 178.7 -> 228.5 mm, vias 5 -> 7
- net /IO Expander/COL7: track 275.7 -> 322.7 mm
- net /IO Expander/COL9: track 227.2 -> 270.3 mm
- net /IO Expander/COL10: track 234.1 -> 227.2 mm, vias 7 -> 6
- net /IO Expander/COL11: track 228.5 -> 234.1 mm
- net /IO Expander/COL8: track 270.3 -> 275.7 mm
